Commit message: penambahan dashboard

File: src/Delivery_AMR_description/urdf/Delivery_AMR.xacro (robot description, xacro)
@@ -168,5 +168,5 @@
   <parent link="base_link"/>
   <child link="right_wheel_1"/>
-  <axis xyz="0.0 -1.0 0.0"/>
+  <axis xyz="0.0 1.0 0.0"/>
 </joint>
 <joint name="Revolute 6" type="continuous">
@@ -174,5 +174,5 @@
   <parent link="base_link"/>
   <child link="left_wheel_1"/>
-  <axis xyz="0.0 -1.0 0.0"/>
+  <axis xyz="0.0 1.0 0.0"/>
 </joint>
 <!-- BASE FOOTPRINT (Agar robot tidak tenggelam di lantai Gazebo) -->

Commit message: view_robot

File: src/Delivery_AMR_description/urdf/Delivery_AMR.xacro (robot description, xacro)
@@ -180,6 +180,6 @@
 <joint name="base_footprint_joint" type="fixed">
   <origin xyz="0 0 0" rpy="0 0 0" />
-  <parent link="base_footprint" />
-  <child link="base_link" />
+  <parent link="base_link" />
+  <child link="base_footprint" />
 </joint>
 <!-- DUMMY LINK KAMERA -->
